Commit message: Add side camera, resize/retune apple collision, tune grasp geometry
Adds a fixed side-view camera and ROS bridge topic for observing grasp
attempts. Reworks apple_05's collision shape to match its true visual
mesh size (previous shape was oversized, causing premature contact
detection) and retunes mass/inertia accordingly; applies the same
scale fix across the other apple models. Updates the dexhand/UR5e
xacros and launch file for the current grasp pipeline.

Co-Authored-By: Claude Sonnet 5 <noreply@anthropic.com>

File: src/dexhandv2_description/urdf/dexhandv2_right.xacro (robot description, xacro)
@@ -188,5 +188,5 @@
     <origin xyz="-0.00031356817587347915 -0.0028006513879080056 0.007069716391178871" rpy="0 0 0"/>
     <mass value="0.018995895295817036"/>
-    <inertia ixx="1e-06" iyy="1e-06" izz="0.0" ixy="-0.0" iyz="-0.0" ixz="0.0"/>
+    <inertia ixx="1e-06" iyy="1e-06" izz="1e-06" ixy="-0.0" iyz="-0.0" ixz="0.0"/>
   </inertial>
   <visual>
@@ -208,5 +208,5 @@
     <origin xyz="-0.00010202212506613302 -0.002820062193980945 0.007067870395751047" rpy="0 0 0"/>
     <mass value="0.018995895295817036"/>
-    <inertia ixx="1e-06" iyy="1e-06" izz="0.0" ixy="0.0" iyz="-0.0" ixz="0.0"/>
+    <inertia ixx="1e-06" iyy="1e-06" izz="1e-06" ixy="0.0" iyz="-0.0" ixz="0.0"/>
   </inertial>
   <visual>
@@ -228,5 +228,5 @@
     <origin xyz="0.00011862144140123952 -0.0028181864528833943 0.007068122192193688" rpy="0 0 0"/>
     <mass value="0.018995895295817036"/>
-    <inertia ixx="1e-06" iyy="1e-06" izz="0.0" ixy="0.0" iyz="0.0" ixz="0.0"/>
+    <inertia ixx="1e-06" iyy="1e-06" izz="1e-06" ixy="0.0" iyz="0.0" ixz="0.0"/>
   </inertial>
   <visual>
@@ -248,5 +248,5 @@
     <origin xyz="0.0005552836495658926 -0.002793482086718077 0.007056916444342365" rpy="0 0 0"/>
     <mass value="0.018995895295817036"/>
-    <inertia ixx="1e-06" iyy="1e-06" izz="0.0" ixy="0.0" iyz="0.0" ixz="0.0"/>
+    <inertia ixx="1e-06" iyy="1e-06" izz="1e-06" ixy="0.0" iyz="0.0" ixz="0.0"/>
   </inertial>
   <visual>
@@ -268,5 +268,5 @@
     <origin xyz="-0.005783732642998508 -0.005234605010581522 0.005230813563652258" rpy="0 0 0"/>
     <mass value="0.010139940256668681"/>
-    <inertia ixx="0.0" iyy="0.0" izz="0.0" ixy="-0.0" iyz="0.0" ixz="0.0"/>
+    <inertia ixx="1e-06" iyy="1e-06" izz="1e-06" ixy="-0.0" iyz="0.0" ixz="0.0"/>
   </inertial>
   <visual>

File: src/my_pick_and_place/urdf/ur5e_dexhand.xacro (robot description, xacro)
@@ -20,11 +20,19 @@
     <visual>
       <origin xyz="0 0 0.16" rpy="0 0 0"/>
-      <geometry><box size="0.8 0.6 0.25"/></geometry>
+      <geometry><box size="0.36 0.36 0.25"/></geometry>
       <material name="chassis_dark"><color rgba="0.2 0.2 0.2 1.0"/></material>
     </visual>
-    <collision>
-      <origin xyz="0 0 0.16" rpy="0 0 0"/>
-      <geometry><box size="0.8 0.6 0.25"/></geometry>
-    </collision>
+    <!-- Collision deliberately omitted: the UR arm is mounted directly on
+         top of this box (parent="mobile_base_link", z=0.285, right at the
+         box's own top surface), and depending on shoulder_lift/elbow angle
+         the upper arm link can swing down into the box's volume, confirmed
+         live: it visually clipped through the chassis during a grasp
+         descend. ikpy's IK has no self-collision awareness, so nothing
+         stops it from choosing such a configuration, and Gazebo's physics
+         would otherwise fight the resulting overlap with contact forces, a
+         real source of unwanted disturbance during exactly the grasp
+         motions this project is trying to stabilize. The box stays visible
+         (visual kept) and still contributes its mass/inertia for base
+         stability; it just can't physically collide with anything anymore. -->
     <inertial>
       <mass value="100.0"/>
@@ -46,5 +54,12 @@
   </link>
   <joint name="left_wheel_joint" type="continuous">
-    <parent link="mobile_base_link"/><child link="left_wheel"/><origin xyz="0 0.33 0.12" rpy="0 0 0"/><axis xyz="0 1 0"/>
+    <parent link="mobile_base_link"/><child link="left_wheel"/><origin xyz="0 0.20 0.12" rpy="0 0 0"/><axis xyz="0 1 0"/>
+    <!-- Never actively driven (nothing publishes /cmd_vel), so without
+         friction/damping this is a frictionless bearing: any external
+         disturbance (e.g. a bad arm move) can set the whole mobile base
+         rolling or tipping. Kept "continuous" (not "fixed") so the DiffDrive
+         plugin below, which also publishes the odom to base_footprint TF the
+         whole grasp pipeline relies on, still initializes correctly. -->
+    <dynamics damping="50.0" friction="20.0"/>
   </joint>
   <link name="right_wheel">
@@ -54,5 +69,6 @@
   </link>
   <joint name="right_wheel_joint" type="continuous">
-    <parent link="mobile_base_link"/><child link="right_wheel"/><origin xyz="0 -0.33 0.12" rpy="0 0 0"/><axis xyz="0 1 0"/>
+    <parent link="mobile_base_link"/><child link="right_wheel"/><origin xyz="0 -0.20 0.12" rpy="0 0 0"/><axis xyz="0 1 0"/>
+    <dynamics damping="50.0" friction="20.0"/>
   </joint>
   <link name="caster_front">
@@ -62,5 +78,5 @@
   </link>
   <joint name="caster_front_joint" type="fixed">
-    <parent link="mobile_base_link"/><child link="caster_front"/><origin xyz="0.3 0 0.06" rpy="0 0 0"/>
+    <parent link="mobile_base_link"/><child link="caster_front"/><origin xyz="0.16 0 0.06" rpy="0 0 0"/>
   </joint>
   <link name="caster_back">
@@ -70,5 +86,5 @@
   </link>
   <joint name="caster_back_joint" type="fixed">
-    <parent link="mobile_base_link"/><child link="caster_back"/><origin xyz="-0.3 0 0.06" rpy="0 0 0"/>
+    <parent link="mobile_base_link"/><child link="caster_back"/><origin xyz="-0.16 0 0.06" rpy="0 0 0"/>
   </joint>
   <!-- Include UR Robot with Horizontal Arm Pose -->
@@ -154,5 +170,5 @@
       <left_joint>left_wheel_joint</left_joint>
       <right_joint>right_wheel_joint</right_joint>
-      <wheel_separation>0.66</wheel_separation>
+      <wheel_separation>0.40</wheel_separation>
       <wheel_radius>0.12</wheel_radius>
       <odom_publish_frequency>50</odom_publish_frequency>
@@ -172,4 +188,5 @@
       <state_interface name="position"/>
       <state_interface name="velocity"/>
+      <state_interface name="effort"/>
     </joint>
     <joint name="R_Middle_Pitch">
@@ -177,4 +194,5 @@
       <state_interface name="position"/>
       <state_interface name="velocity"/>
+      <state_interface name="effort"/>
     </joint>
     <joint name="R_Ring_Pitch">
@@ -182,4 +200,5 @@
       <state_interface name="position"/>
       <state_interface name="velocity"/>
+      <state_interface name="effort"/>
     </joint>
     <joint name="R_Pinky_Pitch">
@@ -187,4 +206,5 @@
       <state_interface name="position"/>
       <state_interface name="velocity"/>
+      <state_interface name="effort"/>
     </joint>
     <joint name="R_Index_Flexor">
@@ -192,4 +212,5 @@
       <state_interface name="position"/>
       <state_interface name="velocity"/>
+      <state_interface name="effort"/>
     </joint>
     <joint name="R_Middle_Flexor">
@@ -197,4 +218,5 @@
       <state_interface name="position"/>
       <state_interface name="velocity"/>
+      <state_interface name="effort"/>
     </joint>
     <joint name="R_Ring_Flexor">
@@ -202,4 +224,5 @@
       <state_interface name="position"/>
       <state_interface name="velocity"/>
+      <state_interface name="effort"/>
     </joint>
     <joint name="R_Pinky_Flexor">
@@ -207,4 +230,5 @@
       <state_interface name="position"/>
       <state_interface name="velocity"/>
+      <state_interface name="effort"/>
     </joint>
     <joint name="R_Index_DIP">
@@ -212,4 +236,5 @@
       <state_interface name="position"/>
       <state_interface name="velocity"/>
+      <state_interface name="effort"/>
     </joint>
     <joint name="R_Middle_DIP">
@@ -217,4 +242,5 @@
       <state_interface name="position"/>
       <state_interface name="velocity"/>
+      <state_interface name="effort"/>
     </joint>
     <joint name="R_Ring_DIP">
@@ -222,4 +248,5 @@
       <state_interface name="position"/>
       <state_interface name="velocity"/>
+      <state_interface name="effort"/>
     </joint>
     <joint name="R_Pinky_DIP">
@@ -227,4 +254,5 @@
       <state_interface name="position"/>
       <state_interface name="velocity"/>
+      <state_interface name="effort"/>
     </joint>
     <joint name="R_Thumb_Yaw">
@@ -232,4 +260,5 @@
       <state_interface name="position"/>
       <state_interface name="velocity"/>
+      <state_interface name="effort"/>
     </joint>
     <joint name="R_Thumb_Roll">
@@ -237,4 +266,5 @@
       <state_interface name="position"/>
       <state_interface name="velocity"/>
+      <state_interface name="effort"/>
     </joint>
     <joint name="R_Thumb_Flexor">
@@ -242,4 +272,5 @@
       <state_interface name="position"/>
       <state_interface name="velocity"/>
+      <state_interface name="effort"/>
     </joint>
     <joint name="R_Thumb_DIP">
@@ -247,4 +278,5 @@
       <state_interface name="position"/>
       <state_interface name="velocity"/>
+      <state_interface name="effort"/>
     </joint>
     <joint name="R_Index_Yaw">
@@ -252,4 +284,5 @@
       <state_interface name="position"/>
       <state_interface name="velocity"/>
+      <state_interface name="effort"/>
     </joint>
     <joint name="R_Middle_Yaw">
@@ -257,4 +290,5 @@
       <state_interface name="position"/>
       <state_interface name="velocity"/>
+      <state_interface name="effort"/>
     </joint>
     <joint name="R_Ring_Yaw">
@@ -262,4 +296,5 @@
       <state_interface name="position"/>
       <state_interface name="velocity"/>
+      <state_interface name="effort"/>
     </joint>
     <joint name="R_Pinky_Yaw">
@@ -267,4 +302,5 @@
       <state_interface name="position"/>
       <state_interface name="velocity"/>
+      <state_interface name="effort"/>
     </joint>
     <joint name="R_Thumb_Pitch">
@@ -272,4 +308,5 @@
       <state_interface name="position"/>
       <state_interface name="velocity"/>
+      <state_interface name="effort"/>
     </joint>
   </ros2_control>
